File: hardware/_saved_can-display.sch (KiCad schematic (older format))
At the start: 31 parts, among them J1 Conn_01x10_Female, J2 Conn_02x09_Odd_Even, J3 Conn_01x04_Male, J4 Conn_01x02_Male, J5 Conn_01x04_Male, J6 Conn_01x04_Male, U1 STM32F446RCTx, U2 MCP4019, U3 TLC59284, U4 MCP2562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

Commit message: schematic and route f4
Parts:
- gave numbers to parts that had none: 1
Changed lines of the file:
@@
 NoConn ~ 7400 12250
 $Comp
-L C C?
+L C C8
 U 1 1 5AC72FE5
 P 6100 850
-F 0 "C?" H 6125 950 50  0000 L CNN
+F 0 "C8" H 6125 950 50  0000 L CNN
 F 1 "0.1uF" H 6125 750 50  0000 L CNN
 F 2 "Capacitors_SMD:C_0603" H 6138 700 50  0001 C CNN
@@
 $EndComp
 $Comp
-L +3.3V #PWR?
+L +3.3V #PWR045
 U 1 1 5AC72FEB
 P 6100 700
-F 0 "#PWR?" H 6100 550 50  0001 C CNN
+F 0 "#PWR045" H 6100 550 50  0001 C CNN
 F 1 "+3.3V" H 6100 840 50  0000 C CNN
 F 2 "" H 6100 700 50  0001 C CNN
@@
 $EndComp
 $Comp
-L GND #PWR?
+L GND #PWR046
 U 1 1 5AC72FF1
 P 6100 1000
-F 0 "#PWR?" H 6100 750 50  0001 C CNN
+F 0 "#PWR046" H 6100 750 50  0001 C CNN
 F 1 "GND" H 6100 850 50  0000 C CNN
 F 2 "" H 6100 1000 50  0001 C CNN

Commit message: add vcap_1
Parts:
- added C11: 4.7uF, Capacitors_SMD:C_0603, symbol C
Connections:
- net GND: now also C11.2
- net at U1.30 (VCAP_1): now also C11.1
Changed lines of the file:
@@
 	1    0    0    -1
 $EndComp
+$Comp
+L C C11
+U 1 1 5AC71785
+P 7150 10700
+F 0 "C11" H 7175 10800 50  0000 L CNN
+F 1 "4.7uF" H 7175 10600 50  0000 L CNN
+F 2 "Capacitors_SMD:C_0603" H 7188 10550 50  0001 C CNN
+F 3 "" H 7150 10700 50  0001 C CNN
+	1    7150 10700
+	1    0    0    -1
+$EndComp
+$Comp
+L GND #PWR047
+U 1 1 5AC71B4B
+P 7150 10950
+F 0 "#PWR047" H 7150 10700 50  0001 C CNN
+F 1 "GND" H 7150 10800 50  0000 C CNN
+F 2 "" H 7150 10950 50  0001 C CNN
+F 3 "" H 7150 10950 50  0001 C CNN
+	1    7150 10950
+	1    0    0    -1
+$EndComp
+Wire Wire Line
+	7150 10950 7150 10850
+Wire Wire Line
+	7150 10550 7150 10450
+Wire Wire Line
+	7150 10450 7400 10450
 $EndSCHEMATC
