File: hardware/can-display.kicad_pcb (KiCad board)
At the start: 4 copper layers, 35.6 x 29.2 mm, 30 parts, among them J1 Conn_01x10_Female, J2 Conn_02x09_Odd_Even, J3 Conn_01x04_Male, J4 Conn_01x02_Male, J5 Conn_01x04_Male, J6 Conn_01x04_Male, U1 STM32F072C8Tx, U2 MCP4019, U3 TLC59284, U4 MCP2562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

Commit message: schematic and route f4
Parts:
- added C8: 0.1uF, Capacitors_SMD:C_0603, B.Cu at (49.0, 49.0)
- C5: moved to F.Cu
- U1: value STM32F072C8Tx -> STM32F446RCTx; footprint Housings_QFP:LQFP-48_7x7mm_Pitch0.5mm -> Housings_QFP:LQFP-64_10x10mm_Pitch0.5mm
- moved J6 4.83 mm to (34.3, 49.5)
- moved C3 2.90 mm to (51.1, 35.6)
- moved C2 2.82 mm to (53.3, 42.5)
- moved R2 2.04 mm to (53.7, 39.6)
- moved C5 1.37 mm to (52.1, 44.7), turned to 90 degrees
- moved U1 1.14 mm to (45.7, 41.7)
- moved R5 1.14 mm to (28.4, 46.2)
- moved C4 1.13 mm to (38.4, 38.4)
- moved R6 1.05 mm to (32.0, 46.2)
- moved J5 0.77 mm to (35.6, 43.7)
- moved C1 0.57 mm to (39.9, 47.2), turned to 0 degrees
- moved R7 0.18 mm to (46.4, 38.0)
Connections:
- U1 pad 11: OLED_SDCS -> (no net)
- U1 pad 12: OLED_OCS -> GND
- U1 pad 13: OLED_RST -> +3V3
- U1 pad 14: OLED_DC -> OLED_SDCS
- U1 pad 15: OLED_SCK -> OLED_OCS
- U1 pad 16: OLED_MISO -> OLED_RST
- U1 pad 17: OLED_MOSI -> OLED_DC
- U1 pad 18: ADC_KNOB -> GND
- U1 pad 19: ADC_KNOB2 -> +3V3
- U1 pad 20: (no net) -> OLED_SCK
- U1 pad 21: (no net) -> OLED_MISO
- U1 pad 22: (no net) -> OLED_MOSI
- U1 pad 23: GND -> (no net)
- U1 pad 24: +3V3 -> (no net)
- U1 pad 25: LED_LAT -> (no net)
- U1 pad 26: LED_SCK -> ADC_KNOB
- U1 pad 27: (no net) -> ADC_KNOB2
- U1 pad 28: LED_MOSI -> (no net)
- U1 pad 31: (no net) -> GND
- U1 pad 32: (no net) -> +3V3
- U1 pad 33: (no net) -> LED_LAT
- U1 pad 34: Net-(J6-Pad4) -> LED_SCK
- U1 pad 35: GND -> (no net)
- U1 pad 36: +3V3 -> LED_MOSI
- U1 pad 37: Net-(J6-Pad2) -> (no net)
- U1 pad 39: DRIVER_1 -> (no net)
- U1 pad 40: DRIVER_2 -> (no net)
- U1 pad 42: SCL -> (no net)
- U1 pad 43: SDA -> (no net)
- U1 pad 44: Net-(R7-Pad1) -> (no net)
- U1 pad 45: CAN_RX -> (no net)
- U1 pad 46: CAN_TX -> Net-(J6-Pad4)
- U1 pad 8: GND -> (no net)
- U1 pad 9: +3V3 -> (no net)
Routing:
- net SDA: track 31.0 -> 15.4 mm, vias 3 -> 2
- net SCL: track 32.8 -> 18.7 mm, vias 1 -> 3
- net CAN_TX: track 18.1 -> 27.9 mm
- net +3V3: track 17.9 -> 26.3 mm, vias 6 -> 8
- net GND: track 48.2 -> 56.4 mm, vias 17 -> 16
- net Net-(J6-Pad2): track 13.7 -> 19.2 mm, vias 1 -> 2
- net OLED_RST: track 8.01 -> 12.4 mm
- net OLED_DC: track 8.50 -> 11.7 mm, vias 0 -> 1
- net +12V: track 31.3 -> 33.9 mm
- net OLED_SCK: track 10.4 -> 12.6 mm
- net Net-(J6-Pad4): track 13.4 -> 15.0 mm
- net OLED_SDCS: track 9.42 -> 10.7 mm
- net OLED_OCS: track 10.2 -> 11.2 mm
- net LED_SCK: track 14.1 -> 14.9 mm
- net ADC_KNOB2: track 19.8 -> 20.6 mm, vias 2 -> 1
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
Commit message: add vcap_1
Parts:
- added C11: 4.7uF, Capacitors_SMD:C_0603, F.Cu at (41.4, 47.5)
Connections:
- U1 pad 30: (no net) -> Net-(C11-Pad1)
Routing:
- net Net-(C11-Pad1): track 0.00 -> 2.35 mm, vias 0 -> 1
- net ADC_KNOB: track 16.1 -> 16.6 mm
Changed lines of the file:
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@@
 (kicad_pcb (version 4) (host pcbnew 4.0.7)
   (general
-    (links 112)
-    (no_connects 0)
+    (links 114)
+    (no_connects 2)
     (area 25.324999 25.324999 61.035001 54.685001)
     (thickness 1.6)
     (drawings 8)
-    (tracks 563)
+    (tracks 571)
     (zones 0)
-    (modules 31)
-    (nets 49)
+    (modules 32)
+    (nets 50)
   )
   (page A4)
@@
   (net 47 OLED_SDCS)
   (net 48 OLED_MISO)
+  (net 49 "Net-(C11-Pad1)")
   (net_class Default "This is the default net class."
     (clearance 0.2032)
@@
     (add_net LED_MOSI)
     (add_net LED_SCK)
+    (add_net "Net-(C11-Pad1)")
     (add_net "Net-(D1-Pad2)")
     (add_net "Net-(J2-Pad10)")
@@
     (pad 28 smd rect (at 1.75 -5.7 90) (size 1 0.25) (layers B.Cu B.Paste B.Mask))
     (pad 29 smd rect (at 2.25 -5.7 90) (size 1 0.25) (layers B.Cu B.Paste B.Mask))
-    (pad 30 smd rect (at 2.75 -5.7 90) (size 1 0.25) (layers B.Cu B.Paste B.Mask))
+    (pad 30 smd rect (at 2.75 -5.7 90) (size 1 0.25) (layers B.Cu B.Paste B.Mask)
+      (net 49 "Net-(C11-Pad1)"))
     (pad 31 smd rect (at 3.25 -5.7 90) (size 1 0.25) (layers B.Cu B.Paste B.Mask)
       (net 1 GND))
@@
     (pad 1 smd rect (at -0.75 0) (size 0.8 0.75) (layers B.Cu B.Paste B.Mask)
       (net 2 +3V3))
+    (model Capacitors_SMD.3dshapes/C_0603.wrl
+      (at (xyz 0 0 0))
+      (scale (xyz 1 1 1))
+      (rotate (xyz 0 0 0))
+    )
+  )
+  (module Capacitors_SMD:C_0603 (layer F.Cu)
+    (at 41.402 47.498 180)
+    (descr "Capacitor SMD 0603, reflow soldering, AVX (see smccp.pdf)")
+    (tags "capacitor 0603")
+    (attr smd)
+    (fp_text reference C11 (at 0 -1.5 180) (layer F.SilkS)
+      (effects (font (size 1 1) (thickness 0.15)))
+    )
+    (fp_text value 4.7uF (at 0 1.5 180) (layer F.Fab)
+      (effects (font (size 1 1) (thickness 0.15)))
+    )
+    (fp_line (start 1.4 0.65) (end -1.4 0.65) (layer F.CrtYd) (width 0.05))
+    (fp_line (start 1.4 0.65) (end 1.4 -0.65) (layer F.CrtYd) (width 0.05))
+    (fp_line (start -1.4 -0.65) (end -1.4 0.65) (layer F.CrtYd) (width 0.05))
+    (fp_line (start -1.4 -0.65) (end 1.4 -0.65) (layer F.CrtYd) (width 0.05))
+    (fp_line (start 0.35 0.6) (end -0.35 0.6) (layer F.SilkS) (width 0.12))
+    (fp_line (start -0.35 -0.6) (end 0.35 -0.6) (layer F.SilkS) (width 0.12))
+    (fp_line (start -0.8 -0.4) (end 0.8 -0.4) (layer F.Fab) (width 0.1))
+    (fp_line (start 0.8 -0.4) (end 0.8 0.4) (layer F.Fab) (width 0.1))
+    (fp_line (start 0.8 0.4) (end -0.8 0.4) (layer F.Fab) (width 0.1))
+    (fp_line (start -0.8 0.4) (end -0.8 -0.4) (layer F.Fab) (width 0.1))
+    (fp_text user %R (at 0 0 180) (layer F.Fab)
+      (effects (font (size 0.3 0.3) (thickness 0.075)))
+    )
+    (pad 2 smd rect (at 0.75 0 180) (size 0.8 0.75) (layers F.Cu F.Paste F.Mask)
+      (net 1 GND))
+    (pad 1 smd rect (at -0.75 0 180) (size 0.8 0.75) (layers F.Cu F.Paste F.Mask)
+      (net 49 "Net-(C11-Pad1)"))
     (model Capacitors_SMD.3dshapes/C_0603.wrl
       (at (xyz 0 0 0))
@@
   (via (at 42.545 35.024198) (size 0.4572) (drill 0.3048) (layers F.Cu B.Cu) (net 41))
   (segment (start 41.456 35.318) (end 41.656 35.318) (width 0.2032) (layer F.Cu) (net 41))
+  (segment (start 44.97 47.356) (end 44.97 46.6528) (width 0.2032) (layer B.Cu) (net 42))
+  (segment (start 44.97 46.6528) (end 44.87641 46.55921) (width 0.2032) (layer B.Cu) (net 42))
+  (segment (start 44.87641 46.55921) (end 44.87641 46.48446) (width 0.2032) (layer B.Cu) (net 42))
+  (segment (start 44.87641 46.48446) (end 43.60395 45.212) (width 0.2032) (layer B.Cu) (net 42))
+  (segment (start 42.672 45.212) (end 43.60395 45.212) (width 0.2032) (layer B.Cu) (net 42))
+  (segment (start 38.333289 45.880353) (end 39.001642 45.212) (width 0.2032) (layer F.Cu) (net 42))
+  (segment (start 39.001642 45.212) (end 42.672 45.212) (width 0.2032) (layer F.Cu) (net 42))
+  (via (at 42.672 45.212) (size 0.5842) (drill 0.3556) (layers F.Cu B.Cu) (net 42))
   (segment (start 38.333289 45.880353) (end 37.985642 46.228) (width 0.2032) (layer F.Cu) (net 42))
   (segment (start 37.985642 46.228) (end 32.754 46.228) (width 0.2032) (layer F.Cu) (net 42))
   (segment (start 32.754 46.228) (end 32.754 43.994) (width 0.2032) (layer F.Cu) (net 42))
   (segment (start 32.754 43.994) (end 33.06 43.688) (width 0.2032) (layer F.Cu) (net 42))
-  (segment (start 43.561 45.880353) (end 38.333289 45.880353) (width 0.2032) (layer F.Cu) (net 42))
-  (segment (start 44.97 47.356) (end 44.899801 47.285801) (width 0.2032) (layer B.Cu) (net 42))
-  (segment (start 44.899801 47.285801) (end 44.899801 46.612159) (width 0.2032) (layer B.Cu) (net 42))
-  (segment (start 44.876409 46.484459) (end 44.272303 45.880353) (width 0.2032) (layer B.Cu) (net 42))
-  (segment (start 44.899801 46.612159) (end 44.87641 46.588768) (width 0.2032) (layer B.Cu) (net 42))
-  (segment (start 44.87641 46.588768) (end 44.876409 46.484459) (width 0.2032) (layer B.Cu) (net 42))
-  (segment (start 44.272303 45.880353) (end 43.561 45.880353) (width 0.2032) (layer B.Cu) (net 42))
-  (via (at 43.561 45.880353) (size 0.4572) (drill 0.3048) (layers F.Cu B.Cu) (net 42))
+  (segment (start 42.352658 45.954299) (end 42.346958 45.948599) (width 0.2032) (layer F.Cu) (net 43))
+  (segment (start 42.346958 45.948599) (end 38.839793 45.948599) (width 0.2032) (layer F.Cu) (net 43))
+  (segment (start 38.839793 45.948599) (end 37.544392 47.244) (width 0.2032) (layer F.Cu) (net 43))
+  (segment (start 37.544392 47.244) (end 32.512 47.244) (width 0.2032) (layer F.Cu) (net 43))
+  (segment (start 44.47 47.356) (end 44.47 46.6528) (width 0.2032) (layer B.Cu) (net 43))
+  (segment (start 44.47 46.6528) (end 43.663729 45.846529) (width 0.2032) (layer B.Cu) (net 43))
+  (segment (start 43.663729 45.846529) (end 42.460428 45.846529) (width 0.2032) (layer B.Cu) (net 43))
+  (segment (start 42.460428 45.846529) (end 42.352658 45.954299) (width 0.2032) (layer B.Cu) (net 43))
+  (via (at 42.352658 45.954299) (size 0.5842) (drill 0.3556) (layers F.Cu B.Cu) (net 43))
   (segment (start 32.004 46.736) (end 32.512 47.244) (width 0.2032) (layer F.Cu) (net 43))
-  (segment (start 32.512 47.244) (end 42.116589 47.244) (width 0.2032) (layer F.Cu) (net 43))
   (segment (start 32.004 45.132) (end 32.004 46.736) (width 0.2032) (layer F.Cu) (net 43))
   (segment (start 30.56 43.688) (end 32.004 45.132) (width 0.2032) (layer F.Cu) (net 43))
   (segment (start 29.198 46.228) (end 29.198 45.05) (width 0.2032) (layer F.Cu) (net 43))
   (segment (start 29.198 45.05) (end 30.56 43.688) (width 0.2032) (layer F.Cu) (net 43))
-  (segment (start 42.946836 46.413753) (end 42.116589 47.244) (width 0.2032) (layer F.Cu) (net 43))
-  (segment (start 44.47 47.356) (end 44.47 46.6528) (width 0.2032) (layer B.Cu) (net 43))
-  (segment (start 44.47 46.6528) (end 44.230953 46.413753) (width 0.2032) (layer B.Cu) (net 43))
-  (segment (start 44.230953 46.413753) (end 42.946836 46.413753) (width 0.2032) (layer B.Cu) (net 43))
-  (via (at 42.946836 46.413753) (size 0.4572) (drill 0.3048) (layers F.Cu B.Cu) (net 43))
   (segment (start 44.449547 38.769706) (end 41.637621 41.581632) (width 0.2032) (layer B.Cu) (net 44))
   (segment (start 41.63762 45.14108) (end 40.830101 45.948599) (width 0.2032) (layer B.Cu) (net 44))
@@
   (segment (start 47.241398 46.424198) (end 45.466 46.424198) (width 0.2032) (layer B.Cu) (net 48))
   (via (at 45.466 46.424198) (size 0.4572) (drill 0.3048) (layers F.Cu B.Cu) (net 48))
+  (segment (start 42.97 47.356) (end 42.97 46.502406) (width 0.2032) (layer B.Cu) (net 49))
+  (segment (start 42.97 46.502406) (end 43.028976 46.44343) (width 0.2032) (layer B.Cu) (net 49))
+  (segment (start 42.152 47.498) (end 42.152 47.320406) (width 0.2032) (layer F.Cu) (net 49))
+  (segment (start 42.152 47.320406) (end 43.028976 46.44343) (width 0.2032) (layer F.Cu) (net 49))
+  (via (at 43.028976 46.44343) (size 0.5842) (drill 0.3556) (layers F.Cu B.Cu) (net 49))
   (zone (net 1) (net_name GND) (layer GND.Cu) (hatch edge 0.508)
     (connect_pads (clearance 0.2032))

Commit message: Switch to F336RET6
Parts:
- U1: value STM32F446RCTx -> STM32F446RETx
Changed lines of the file:
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@@
   (general
     (links 114)
-    (no_connects 2)
+    (no_connects 1)
     (area 25.324999 25.324999 61.035001 54.685001)
     (thickness 1.6)
@@
       (effects (font (size 1 1) (thickness 0.15)) (justify mirror))
     )
-    (fp_text value STM32F446RCTx (at 0 -7.2 180) (layer B.Fab)
-      (effects (font (size 1 1) (thickness 0.15)) (justify mirror))
-    )
+    (fp_text value STM32F446RETx (at 0 -7.2 180) (layer B.Fab)
+      (effects (font (size 1 1) (thickness 0.15)) (justify mirror))
+    )
