File: hardware/can-display.kicad_pcb (KiCad board)
At the start: 4 copper layers, 35.6 x 29.2 mm, 32 parts, among them J1 Conn_01x10_Female, J2 Conn_02x09_Odd_Even, J3 Conn_01x04_Male, J4 Conn_01x02_Male, J5 Conn_01x04_Male, J6 Conn_01x04_Male, U1 STM32F446RETx, U2 MCP4019, U3 TLC59284, U4 MCP2562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

Commit message: Add i2c resistors
Parts:
- added R8: 4.7k, Resistors_SMD:R_0603, F.Cu at (34.0, 32.3)
- added R9: 4.7k, Resistors_SMD:R_0603, F.Cu at (33.8, 28.4)
Routing:
- net +3V3: track 26.3 -> 30.8 mm, vias 8 -> 9
- net SDA: track 15.4 -> 18.7 mm, vias 2 -> 3
- net SCL: track 18.7 -> 19.3 mm
Changed lines of the file:
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@@
 (kicad_pcb (version 4) (host pcbnew 4.0.7)
   (general
-    (links 114)
-    (no_connects 1)
+    (links 118)
+    (no_connects 4)
     (area 25.324999 25.324999 61.035001 54.685001)
     (thickness 1.6)
     (drawings 8)
-    (tracks 571)
+    (tracks 586)
     (zones 0)
-    (modules 32)
+    (modules 34)
     (nets 50)
   )
@@
     (tags "resistor 0603")
     (attr smd)
-    (fp_text reference R1 (at -2.236226 0.054084) (layer F.SilkS)
+    (fp_text reference R1 (at 0.049774 1.324084) (layer F.SilkS)
       (effects (font (size 1 1) (thickness 0.15)))
     )
@@
       (net 49 "Net-(C11-Pad1)"))
     (model Capacitors_SMD.3dshapes/C_0603.wrl
+      (at (xyz 0 0 0))
+      (scale (xyz 1 1 1))
+      (rotate (xyz 0 0 0))
+    )
+  )
+  (module Resistors_SMD:R_0603 (layer F.Cu)
+    (at 34.036 32.258 180)
+    (descr "Resistor SMD 0603, reflow soldering, Vishay (see dcrcw.pdf)")
+    (tags "resistor 0603")
+    (attr smd)
+    (fp_text reference R8 (at 2.286 0 180) (layer F.SilkS)
+      (effects (font (size 1 1) (thickness 0.15)))
+    )
+    (fp_text value 4.7k (at 0 1.5 180) (layer F.Fab)
+      (effects (font (size 1 1) (thickness 0.15)))
+    )
+    (fp_text user %R (at 0 0 180) (layer F.Fab)
+      (effects (font (size 0.4 0.4) (thickness 0.075)))
+    )
+    (fp_line (start -0.8 0.4) (end -0.8 -0.4) (layer F.Fab) (width 0.1))
+    (fp_line (start 0.8 0.4) (end -0.8 0.4) (layer F.Fab) (width 0.1))
+    (fp_line (start 0.8 -0.4) (end 0.8 0.4) (layer F.Fab) (width 0.1))
+    (fp_line (start -0.8 -0.4) (end 0.8 -0.4) (layer F.Fab) (width 0.1))
+    (fp_line (start 0.5 0.68) (end -0.5 0.68) (layer F.SilkS) (width 0.12))
+    (fp_line (start -0.5 -0.68) (end 0.5 -0.68) (layer F.SilkS) (width 0.12))
+    (fp_line (start -1.25 -0.7) (end 1.25 -0.7) (layer F.CrtYd) (width 0.05))
+    (fp_line (start -1.25 -0.7) (end -1.25 0.7) (layer F.CrtYd) (width 0.05))
+    (fp_line (start 1.25 0.7) (end 1.25 -0.7) (layer F.CrtYd) (width 0.05))
+    (fp_line (start 1.25 0.7) (end -1.25 0.7) (layer F.CrtYd) (width 0.05))
+    (pad 1 smd rect (at -0.75 0 180) (size 0.5 0.9) (layers F.Cu F.Paste F.Mask)
+      (net 29 SCL))
+    (pad 2 smd rect (at 0.75 0 180) (size 0.5 0.9) (layers F.Cu F.Paste F.Mask)
+      (net 2 +3V3))
+    (model ${KISYS3DMOD}/Resistors_SMD.3dshapes/R_0603.wrl
+      (at (xyz 0 0 0))
+      (scale (xyz 1 1 1))
+      (rotate (xyz 0 0 0))
+    )
+  )
+  (module Resistors_SMD:R_0603 (layer F.Cu)
+    (at 33.782 28.448 180)
+    (descr "Resistor SMD 0603, reflow soldering, Vishay (see dcrcw.pdf)")
+    (tags "resistor 0603")
+    (attr smd)
+    (fp_text reference R9 (at 2.032 0 180) (layer F.SilkS)
+      (effects (font (size 1 1) (thickness 0.15)))
+    )
+    (fp_text value 4.7k (at 0 1.5 180) (layer F.Fab)
+      (effects (font (size 1 1) (thickness 0.15)))
+    )
+    (fp_text user %R (at 0 0 180) (layer F.Fab)
+      (effects (font (size 0.4 0.4) (thickness 0.075)))
+    )
+    (fp_line (start -0.8 0.4) (end -0.8 -0.4) (layer F.Fab) (width 0.1))
+    (fp_line (start 0.8 0.4) (end -0.8 0.4) (layer F.Fab) (width 0.1))
+    (fp_line (start 0.8 -0.4) (end 0.8 0.4) (layer F.Fab) (width 0.1))
+    (fp_line (start -0.8 -0.4) (end 0.8 -0.4) (layer F.Fab) (width 0.1))
+    (fp_line (start 0.5 0.68) (end -0.5 0.68) (layer F.SilkS) (width 0.12))
+    (fp_line (start -0.5 -0.68) (end 0.5 -0.68) (layer F.SilkS) (width 0.12))
+    (fp_line (start -1.25 -0.7) (end 1.25 -0.7) (layer F.CrtYd) (width 0.05))
+    (fp_line (start -1.25 -0.7) (end -1.25 0.7) (layer F.CrtYd) (width 0.05))
+    (fp_line (start 1.25 0.7) (end 1.25 -0.7) (layer F.CrtYd) (width 0.05))
+    (fp_line (start 1.25 0.7) (end -1.25 0.7) (layer F.CrtYd) (width 0.05))
+    (pad 1 smd rect (at -0.75 0 180) (size 0.5 0.9) (layers F.Cu F.Paste F.Mask)
+      (net 30 SDA))
+    (pad 2 smd rect (at 0.75 0 180) (size 0.5 0.9) (layers F.Cu F.Paste F.Mask)
+      (net 2 +3V3))
+    (model ${KISYS3DMOD}/Resistors_SMD.3dshapes/R_0603.wrl
       (at (xyz 0 0 0))
       (scale (xyz 1 1 1))
@@
   (segment (start 39.637726 31.865718) (end 39.594924 31.822916) (width 0.3048) (layer F.Cu) (net 1))
   (via (at 39.594924 31.822916) (size 0.5842) (drill 0.3556) (layers F.Cu B.Cu) (net 1))
+  (segment (start 33.032 28.448) (end 33.032 28.648) (width 0.2032) (layer F.Cu) (net 2))
+  (segment (start 34.036 30.156711) (end 34.036 30.48) (width 0.2032) (layer F.Cu) (net 2))
+  (segment (start 33.032 28.648) (end 34.036 29.652) (width 0.2032) (layer F.Cu) (net 2))
+  (segment (start 34.036 29.652) (end 34.036 30.156711) (width 0.2032) (layer F.Cu) (net 2))
+  (segment (start 33.286 32.258) (end 33.286 32.058) (width 0.2032) (layer F.Cu) (net 2))
+  (segment (start 33.286 32.058) (end 34.036 31.308) (width 0.2032) (layer F.Cu) (net 2))
+  (segment (start 34.036 31.308) (end 34.036 30.48) (width 0.2032) (layer F.Cu) (net 2))
+  (via (at 34.036 30.48) (size 0.4572) (drill 0.3048) (layers F.Cu B.Cu) (net 2))
   (segment (start 39.116 47.244) (end 38.354 48.006) (width 0.2032) (layer B.Cu) (net 2))
   (via (at 38.354 48.006) (size 0.4572) (drill 0.3048) (layers F.Cu B.Cu) (net 2))
@@
   (segment (start 40.142527 33.029115) (end 40.142527 33.742757) (width 0.2032) (layer F.Cu) (net 28))
   (via (at 38.982028 33.782) (size 0.4572) (drill 0.3048) (layers F.Cu B.Cu) (net 28))
+  (segment (start 34.786 32.258) (end 35.433 32.258) (width 0.2032) (layer F.Cu) (net 29))
+  (segment (start 35.433 28.575) (end 35.433 32.258) (width 0.2032) (layer F.Cu) (net 29))
+  (segment (start 35.433 32.258) (end 35.433 32.601332) (width 0.2032) (layer F.Cu) (net 29))
   (segment (start 40.259 34.750719) (end 41.073285 34.750719) (width 0.2032) (layer PWR.Cu) (net 29))
   (segment (start 41.073285 34.750719) (end 41.272967 34.950401) (width 0.2032) (layer PWR.Cu) (net 29))
@@
   (segment (start 36.638226 28.079916) (end 36.235026 28.079916) (width 0.2032) (layer F.Cu) (net 29))
   (segment (start 35.433 32.601332) (end 37.201867 34.370199) (width 0.2032) (layer F.Cu) (net 29))
-  (segment (start 35.433 28.575) (end 35.433 32.601332) (width 0.2032) (layer F.Cu) (net 29))
   (segment (start 44.503203 34.490797) (end 45.714079 34.490797) (width 0.2032) (layer F.Cu) (net 29))
   (segment (start 45.714079 34.490797) (end 45.974 34.750718) (width 0.2032) (layer F.Cu) (net 29))
@@
   (segment (start 46.47 35.246718) (end 45.974 34.750718) (width 0.2032) (layer B.Cu) (net 29))
   (via (at 45.974 34.750718) (size 0.4572) (drill 0.3048) (layers F.Cu B.Cu) (net 29))
+  (segment (start 35.991165 30.515076) (end 34.833076 30.515076) (width 0.2032) (layer B.Cu) (net 30))
+  (segment (start 34.833076 30.515076) (end 34.798 30.48) (width 0.2032) (layer B.Cu) (net 30))
+  (via (at 34.798 30.48) (size 0.4572) (drill 0.3048) (layers F.Cu B.Cu) (net 30))
+  (segment (start 34.532 28.448) (end 34.532 30.214) (width 0.2032) (layer F.Cu) (net 30))
+  (segment (start 34.532 30.214) (end 34.798 30.48) (width 0.2032) (layer F.Cu) (net 30))
   (segment (start 45.974 32.893) (end 46.99 33.909) (width 0.2032) (layer GND.Cu) (net 30))
   (segment (start 46.99 33.909) (end 46.99 34.798) (width 0.2032) (layer GND.Cu) (net 30))

Commit message: board almost final
Parts:
- added C12: 2.2uF, Capacitors_SMD:C_0603, B.Cu at (39.4, 35.6)
- added D2: LED, LEDs:LED_0603_HandSoldering, B.Cu at (57.8, 17.8)
- added D3: LED, LEDs:LED_0603_HandSoldering, B.Cu at (57.8, 20.3)
- added D4: LED, LEDs:LED_0603_HandSoldering, B.Cu at (57.8, 22.9)
- added R10: 1k, Resistors_SMD:R_0603, F.Cu at (54.0, 18.4)
- added R11: 1k, Resistors_SMD:R_0603, F.Cu at (54.0, 21.6)
- added R12: 1k, Resistors_SMD:R_0603, F.Cu at (55.9, 24.1)
- C11: value 4.7uF -> 2.2uF
- R7: moved to B.Cu
- U1: value STM32F446RETx -> STM32F429VITx; footprint Housings_QFP:LQFP-64_10x10mm_Pitch0.5mm -> Housings_QFP:LQFP-100_14x14mm_Pitch0.5mm
- U4: footprint Housings_DFN_QFN:DFN-8-1EP_3x3mm_Pitch0.65mm -> Housings_SOIC:SOIC-8_3.9x4.9mm_Pitch1.27mm
- U7: footprint Housings_DFN_QFN:DFN-8-1EP_6x5mm_Pitch1.27mm_LargeFlag -> Housings_SOIC:SOIC-8_3.9x4.9mm_Pitch1.27mm
- moved D1 28.9 mm to (29.0, 32.5), turned to 180 degrees
- moved R2 22.0 mm to (31.8, 40.1), turned to 180 degrees
- moved J3 21.8 mm to (35.6, 37.5), turned to 180 degrees
- moved C1 20.7 mm to (58.4, 38.1), turned to 90 degrees
- moved C8 20.2 mm to (54.1, 29.5), turned to 180 degrees
- moved C7 15.9 mm to (38.6, 34.5), turned to 270 degrees
- moved C3 14.2 mm to (53.8, 49.5)
- moved U4 13.2 mm to (41.7, 42.7), turned to 180 degrees
- moved R3 11.2 mm to (46.2, 28.4)
- moved R4 11.1 mm to (46.2, 25.9)
- moved U7 11.1 mm to (41.1, 26.9)
- moved R7 10.8 mm to (51.8, 28.7), turned to 90 degrees
- moved R8 10.2 mm to (34.0, 22.1)
- moved C6 10.2 mm to (38.1, 16.5)
- moved J2 10.2 mm to (43.1, 20.1)
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Connections:
- U1 pad 1: (no net) -> Net-(R10-Pad1)
- U1 pad 10: (no net) -> GND
- U1 pad 11: (no net) -> +3V3
- U1 pad 12: GND -> (no net)
- U1 pad 13: +3V3 -> (no net)
- U1 pad 14: OLED_SDCS -> (no net)
- U1 pad 15: OLED_OCS -> (no net)
- U1 pad 16: OLED_RST -> (no net)
- U1 pad 17: OLED_DC -> (no net)
- U1 pad 18: GND -> (no net)
- U1 pad 2: (no net) -> Net-(R11-Pad1)
- U1 pad 20: OLED_SCK -> GND
- U1 pad 21: OLED_MISO -> (no net)
- U1 pad 22: OLED_MOSI -> +3V3
- U1 pad 23: (no net) -> DRIVER_2
- U1 pad 24: (no net) -> OLED_SDCS
- U1 pad 25: (no net) -> OLED_OCS
- U1 pad 26: ADC_KNOB -> OLED_RST
- U1 pad 27: ADC_KNOB2 -> GND
- U1 pad 28: (no net) -> +3V3
- U1 pad 29: (no net) -> OLED_DC
- U1 pad 3: (no net) -> Net-(R12-Pad1)
- U1 pad 30: Net-(C11-Pad1) -> OLED_SCK
- U1 pad 31: GND -> OLED_MISO
- U1 pad 32: +3V3 -> OLED_MOSI
- U1 pad 33: LED_LAT -> (no net)
- U1 pad 34: LED_SCK -> (no net)
- U1 pad 35: (no net) -> ADC_KNOB
- U1 pad 36: LED_MOSI -> ADC_KNOB2
- U1 pad 46: Net-(J6-Pad4) -> (no net)
- U1 pad 47: GND -> (no net)
- U1 pad 48: +3V3 -> (no net)
- U1 pad 49: Net-(J6-Pad2) -> Net-(C11-Pad1)
- U1 pad 50: (no net) -> +3V3
- U1 pad 55: DRIVER_1 -> (no net)
- U1 pad 56: DRIVER_2 -> (no net)
- U1 pad 58: SCL -> (no net)
- U1 pad 59: SDA -> (no net)
- U1 pad 60: Net-(R7-Pad1) -> (no net)
- U1 pad 61: CAN_RX -> (no net)
- U1 pad 62: CAN_TX -> (no net)
- U1 pad 63: GND -> (no net)
- U1 pad 64: +3V3 -> (no net)
Routing:
- net +5V: track 46.6 -> 69.1 mm, vias 5 -> 4
- net DRIVER_2: track 9.09 -> 27.0 mm
- net Net-(R10-Pad1): track 0.00 -> 17.8 mm, vias 0 -> 1
- net CAN_TX: track 27.9 -> 11.6 mm
- net ADC_KNOB: track 16.6 -> 31.7 mm
- net Net-(J4-Pad1): track 2.87 -> 17.8 mm
- net Net-(R11-Pad1): track 0.00 -> 14.4 mm, vias 0 -> 1
- net +12V: track 33.9 -> 19.9 mm, vias 2 -> 0
- net CAN_RX: track 19.4 -> 7.58 mm
- net Net-(R12-Pad1): track 0.00 -> 11.4 mm, vias 0 -> 1
- net SCL: track 19.3 -> 30.1 mm, vias 3 -> 1
- net SDA: track 18.7 -> 29.3 mm, vias 3 -> 2
- net Net-(D1-Pad2): track 2.48 -> 11.2 mm
- net OLED_SCK: track 12.6 -> 18.8 mm, vias 0 -> 1
- net OLED_SDCS: track 10.7 -> 17.0 mm
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Other:
- board size 35.6 x 29.2 mm -> 35.6 x 39.4 mm
